File: Design/PCB/KICAD/MHGC/MHGC.kicad_pcb (KiCad board)
At the start: 2 copper layers, 267 x 45 mm, 43 parts, among them J1 RTCmodulePin, J2 USB_B_Micro, SW1 SW_MIN, SW2 SW_HOUR, U1 ARDUINO_PRO_MINI

Commit message: Completed PCB design
Parts:
- moved D28 128.0 mm to (13.5, 40.5), turned to 180 degrees
- moved D10 124.0 mm to (249.0, 40.5)
- moved D29 120.4 mm to (25.5, 40.5)
- moved R4 114.7 mm to (254.5, 39.4), turned to 270 degrees
- moved J2 114.7 mm to (242.6, 3.81), turned to 180 degrees
- moved D26 111.9 mm to (51.0, 13.5)
- moved D24 106.4 mm to (51.0, 22.5), turned to 180 degrees
- moved R6 104.2 mm to (259.5, 39.4), turned to 270 degrees
- moved D27 102.5 mm to (51.0, 18.0), turned to 180 degrees
- moved D8 101.6 mm to (216.0, 9.00), turned to 180 degrees
- moved RV1 99.6 mm to (228.6, 8.00), turned to 180 degrees
- moved R5 98.9 mm to (264.6, 39.4), turned to 270 degrees
- moved D25 97.2 mm to (51.0, 9.00), turned to 180 degrees
- moved R3 96.4 mm to (240.0, 31.8), turned to 270 degrees
- moved R1 93.3 mm to (240.0, 19.4), turned to 270 degrees
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Connections:
- D19 pad 2: Net-(D13-Pad1) -> Net-(D19-Pad2)
- D20 pad 1: Net-(D13-Pad1) -> Net-(D19-Pad2)
- D21 pad 2: Net-(D13-Pad1) -> Net-(D19-Pad2)
- D22 pad 1: Net-(D13-Pad1) -> Net-(D19-Pad2)
- D23 pad 2: Net-(D13-Pad1) -> Net-(D19-Pad2)
- D24 pad 1: Net-(D13-Pad1) -> Net-(D19-Pad2)
- D3 pad 1: Net-(D13-Pad1) -> Net-(D19-Pad2)
- D31 pad 2: Net-(D13-Pad1) -> Net-(D19-Pad2)
- D4 pad 2: Net-(D13-Pad1) -> Net-(D19-Pad2)
- R4 pad 2: Net-(D13-Pad1) -> Net-(D19-Pad2)
Routing:
- net Net-(D10-Pad2): track 0.00 -> 381.1 mm, vias 0 -> 5
- net Net-(D15-Pad1): track 0.00 -> 315.2 mm, vias 0 -> 8
- net Net-(D13-Pad1): track 0.00 -> 288.6 mm, vias 0 -> 3
- net Net-(D19-Pad2): track 0.00 -> 247.7 mm, vias 0 -> 7
- net Net-(D1-Pad1): track 0.00 -> 226.8 mm
- net GND: track 0.00 -> 170.2 mm, vias 0 -> 1
- net Net-(D1-Pad2): track 0.00 -> 118.5 mm
- net Net-(J1-Pad3): track 0.00 -> 100.9 mm, vias 0 -> 1
- net Net-(SW2-Pad1): track 0.00 -> 100.2 mm, vias 0 -> 1
- net Net-(J1-Pad4): track 0.00 -> 96.5 mm, vias 0 -> 1
- net +5V: track 0.00 -> 96.3 mm, vias 0 -> 1
- net Net-(SW1-Pad1): track 0.00 -> 76.3 mm, vias 0 -> 1
- net Net-(RV1-Pad2): track 0.00 -> 42.3 mm
- net Net-(D11-Pad1): track 0.00 -> 39.1 mm
- net Net-(J2-Pad6): track 0.00 -> 12.4 mm
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Other:
- board text added: "GOGOMAKER's First PCB mood_HanClock"
- board text added: "Powered by Arduino"

Commit message: Change design files 디자인 파일 중에서, PCB설계에 맞추어 버튼 및 기타 부품이 배치될 공간을 작업하고, 아크릴 관련 공차 설정도 다시 하였다.
Parts:
- J2: footprint Connector_USB:USB_Micro-B_Amphenol_10118194_Horizontal -> 3216LED:USB_Micro-B_Amphenol_10118194_Horizontal
- moved R5 2.54 mm to (264.6, 41.9)
- moved J2 1.36 mm to (241.3, 4.30)
- moved R6 1.27 mm to (259.5, 40.6)
- moved RV1 1.27 mm to (227.3, 8.00)
Connections:
- D19 pad 2: Net-(D19-Pad2) -> Net-(D11-Pad1)
- D20 pad 1: Net-(D19-Pad2) -> Net-(D11-Pad1)
- D21 pad 2: Net-(D19-Pad2) -> Net-(D11-Pad1)
- D22 pad 1: Net-(D19-Pad2) -> Net-(D11-Pad1)
- D23 pad 2: Net-(D19-Pad2) -> Net-(D11-Pad1)
- D24 pad 1: Net-(D19-Pad2) -> Net-(D11-Pad1)
- D3 pad 1: Net-(D19-Pad2) -> Net-(D11-Pad1)
- D31 pad 2: Net-(D19-Pad2) -> Net-(D11-Pad1)
- D4 pad 2: Net-(D19-Pad2) -> Net-(D11-Pad1)
- R4 pad 2: Net-(D19-Pad2) -> Net-(D11-Pad1)
- U1 pad JP6_2: Net-(U1-PadJP6_2) -> GND
- U1 pad JP6_4: Net-(U1-PadJP6_4) -> +5V
- U1 pad JP7_9: Net-(U1-PadJP7_9) -> GND
Routing:
- net Net-(D11-Pad1): track 39.1 -> 310.9 mm, vias 0 -> 8
- net Net-(D19-Pad2): track 247.7 -> 0.00 mm, vias 7 -> 0
- net Net-(RV1-Pad2): track 42.3 -> 80.8 mm, vias 0 -> 1
- net Net-(D1-Pad2): track 118.5 -> 81.3 mm
- net Net-(J1-Pad4): track 96.5 -> 130.7 mm
- net Net-(J1-Pad3): track 100.9 -> 133.9 mm
- net +5V: track 96.3 -> 118.8 mm
- net Net-(SW1-Pad1): track 76.3 -> 94.6 mm
- net Net-(J2-Pad6): track 12.4 -> 0.00 mm
- net Net-(SW2-Pad1): track 100.2 -> 109.2 mm
- net Net-(D1-Pad1): track 226.8 -> 217.9 mm
- net Net-(D10-Pad2): track 381.1 -> 374.1 mm, vias 5 -> 2
- net GND: track 170.2 -> 167.0 mm
- net Net-(D13-Pad1): track 288.6 -> 285.7 mm, vias 3 -> 4
- net Net-(R5-Pad1): track 4.78 -> 7.32 mm
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Other:
- net class Default: clearance 0.2 -> 0.3; trace_width 0.25 -> 0.4
- rule trace_clearance: 0.2 -> 0.3
- rule trace_min: 0.2 -> 0.4
