File: Design/PCB/KICAD/MHGC/MHGC.sch (KiCad schematic (older format))
At the start: 44 parts

Commit message: Started PCB design 드디어 PCB에 부품 배치를 시작했다
Parts:
- removed D32: LED, symbol Device:LED
- removed R?: R_Variable, symbol Device:R_Variable
- added RV1: POT_BRIGHT, 3216LED:POT_BRIGHT, symbol Device:R_POT
- D1, D10, D11, D12, D13, D14, D15, D16, D17, D18, D19, D2, D20, D21, D22, D23, D24, D25, D26, D27, D28, D29, D3, D30, D31, D4, D5, D6, D7, D8, D9: footprint (none) -> 3216LED:3216LED
- J1: renamed from J?; value Conn_01x04_MountingPin -> RTCmodulePin; footprint (none) -> Connector_PinSocket_2.54mm:PinSocket_1x04_P2.54mm_Vertical
- J2: renamed from J?; footprint (none) -> Connector_USB:USB_Micro-B_Amphenol_10118194_Horizontal
- R1, R2, R3, R4, R5, R6: renamed from R?; value R -> 110; footprint (none) -> 3216LED:3216R
- SW1: renamed from SW?; value SW_DIP_x01 -> SW_MIN; footprint (none) -> 3216LED:KLT_SW
- SW2: renamed from SW?; value SW_DIP_x01 -> SW_HOUR; footprint (none) -> 3216LED:KLT_SW
- U1: renamed from U?; footprint MODULE_ARDUINO_PRO_MINI -> 3216LED:MODULE_ARDUINO_PRO_MINI
Connections:
- net at D1.1 (K): now also D11.2 (A), D12.1 (K), D13.2 (A), D14.1 (K), D15.2 (A), D16.1 (K), D17.2 (A), D18.1 (K), D2.2 (A), R5.2
- net at D1.2 (A): now also D10.1 (K), D2.1 (K), D3.2 (A), D4.1 (K), D5.2 (A), D6.1 (K), D7.2 (A), D8.1 (K), D9.2 (A), R6.2
- net at D3.1 (K): now also D13.1 (K), D14.2 (A), D19.1 (K), D19.2 (A), D20.1 (K), D20.2 (A), D21.2 (A), D22.1 (K), D23.2 (A), D24.1 (K), D25.1 (K), D26.2 (A), D27.1 (K), D28.2 (A), D31.2 (A), D4.2 (A), D5.1 (K), D6.2 (A), R3.2, R4.2
- net at D7.1 (K): now also D15.1 (K), D16.2 (A), D21.1 (K), D22.2 (A), D25.2 (A), D26.1 (K), D29.1 (K), D30.2 (A), D8.2 (A), R2.2
- net at D9.1 (K): now also D10.2 (A), D17.1 (K), D18.2 (A), D23.1 (K), D24.2 (A), D27.2 (A), D28.1 (K), D29.2 (A), D30.1 (K), R1.2
- net at D11.1 (K): now also D12.2 (A)
- net GND: now reaches D31.1 (K)
- net GND: now also J1.1 (Pin_1), J2.5 (GND), SW1.2, SW2.2, U1.JP1_5 (GND), U1.JP1_6 (GND), RV1.3
- net +5V: now reaches U1.JP1_4 (VCC)
- net +5V: now also J1.2 (Pin_2), J2.1 (VBUS), RV1.1
- net at U1.JP2_1 (A4): now also J1.3 (Pin_3)
- net at U1.JP2_2 (A5): now also J1.4 (Pin_4)
- net at U1.JP6_10 (MISO): now also SW1.1
- net at U1.JP6_11 (MOSI): now also R6.1
- net at U1.JP6_12 (D10): now also R5.1
- net at U1.JP6_8 (A0): now also RV1.2
- net at U1.JP6_9 (SCK): now also SW2.1
- net at U1.JP7_1 (D9): now also R4.1
- net at U1.JP7_4 (D6): now also R3.1
- net at U1.JP7_5 (D5): now also R2.1
- net at U1.JP7_7 (D3): now also R1.1
- no-connect marks 0 -> 25
Other:
- moved on the sheet: D1, D10, D11, D12, D13, D14, D15, D16, D17, D18, D19, D2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

Commit message: Completed PCB design
Connections:
- net at D13.1 (K), D14.2 (A), D19.1 (K)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: no longer D19.2 (A), D20.1 (K), D21.2 (A), D22.1 (K), D23.2 (A), D24.1 (K), D3.1 (K), D31.2 (A), D4.2 (A), R4.2
- new net: D19.2 (A), D20.1 (K), D21.2 (A), D22.1 (K), D23.2 (A), D24.1 (K), D3.1 (K), D31.2 (A), D4.2 (A), R4.2
Changed lines of the file:
@@
 Connection ~ 1000 3750
-Wire Wire Line
-	1000 3250 1400 3250
 Wire Wire Line
 	1300 4700 1400 4700
@@
 	1000 3150 1000 2950
 Connection ~ 1000 3350
-Wire Wire Line
-	1000 3350 1000 3250
 Connection ~ 1000 2750
 Wire Wire Line
@@
 Wire Wire Line
 	1300 6600 1300 6700
-Connection ~ 1000 3250
-Wire Wire Line
-	1000 3250 1000 3150
 Connection ~ 1000 4150
 Wire Wire Line
 	1000 4150 1000 3950
-Connection ~ 1400 3250
-Wire Wire Line
-	1400 3250 1400 3450
 Wire Wire Line
 	1300 5000 1300 5200
@@
 	1300 1750 1400 1750
 Connection ~ 1300 1750
-Wire Wire Line
-	1400 1750 1400 3250
 Wire Wire Line
 	1000 1950 1000 1750
@@
 	1300 4150 1300 4300
 NoConn ~ 3750 4350
+Wire Wire Line
+	1000 3150 1000 3350
+Wire Wire Line
+	1400 1750 1400 3450
 $EndSCHEMATC

Commit message: Change design files 디자인 파일 중에서, PCB설계에 맞추어 버튼 및 기타 부품이 배치될 공간을 작업하고, 아크릴 관련 공차 설정도 다시 하였다.
Parts:
- J2: footprint Connector_USB:USB_Micro-B_Amphenol_10118194_Horizontal -> 3216LED:USB_Micro-B_Amphenol_10118194_Horizontal
Connections:
- net +5V: now also U1.JP6_4 (VCC_1)
- net GND: now also U1.JP6_2 (GND_1), U1.JP7_9 (GND_2)
- net at D19.2 (A), D20.1 (K), D21.2 (A)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: now also D11.1 (K), D12.2 (A)
- no-connect marks 25 -> 22
Changed lines of the file:
@@
 F 0 "J2" H 3357 2767 50  0000 C CNN
 F 1 "USB_B_Micro" H 3357 2676 50  0000 C CNN
-F 2 "Connector_USB:USB_Micro-B_Amphenol_10118194_Horizontal" H 3450 2250 50  0001 C CNN
+F 2 "3216LED:USB_Micro-B_Amphenol_10118194_Horizontal" H 3450 2250 50  0001 C CNN
 F 3 "~" H 3450 2250 50  0001 C CNN
 	1    3300 2300
@@
 Wire Wire Line
 	700  7650 700  5400
-$Comp
-L ARDUINO_PRO_MINI:ARDUINO_PRO_MINI U1
-U 1 1 60F56053
-P 3050 5350
-F 0 "U1" H 3050 6717 50  0000 C CNN
-F 1 "ARDUINO_PRO_MINI" H 3050 6626 50  0000 C CNN
-F 2 "3216LED:MODULE_ARDUINO_PRO_MINI" H 3050 5350 50  0001 L BNN
-F 3 "" H 3050 5350 50  0001 L BNN
-F 4 "Manufacturer Recommendations" H 3050 5350 50  0001 L BNN "STANDARD"
-F 5 "N/A" H 3050 5350 50  0001 L BNN "MAXIMUM_PACKAGE_HEIGHT"
-F 6 "SparkFun Electronics" H 3050 5350 50  0001 L BNN "MANUFACTURER"
-F 7 "N/A" H 3050 5350 50  0001 L BNN "PARTREV"
-	1    3050 5350
-	1    0    0    -1
-$EndComp
 Wire Wire Line
 	2000 7650 2100 7650
@@
 L power:+5V #PWR08
 U 1 1 60FB5994
-P 3750 4250
-F 0 "#PWR08" H 3750 4100 50  0001 C CNN
-F 1 "+5V" V 3765 4378 50  0000 L CNN
-F 2 "" H 3750 4250 50  0001 C CNN
-F 3 "" H 3750 4250 50  0001 C CNN
-	1    3750 4250
+P 3850 4250
+F 0 "#PWR08" H 3850 4100 50  0001 C CNN
+F 1 "+5V" V 3865 4378 50  0000 L CNN
+F 2 "" H 3850 4250 50  0001 C CNN
+F 3 "" H 3850 4250 50  0001 C CNN
+	1    3850 4250
 	0    1    1    0
 $EndComp
@@
 	0    -1   -1   0
 $EndComp
-NoConn ~ 3750 6450
-NoConn ~ 3750 6350
 NoConn ~ 3750 5950
 NoConn ~ 3750 5850
@@
 	1000 4150 1000 3950
 Wire Wire Line
-	1300 5000 1300 5200
-Wire Wire Line
 	1000 4150 1000 4400
-Wire Wire Line
-	900  2550 900  6700
 Wire Wire Line
 	1300 6700 900  6700
@@
 Wire Wire Line
 	1300 4150 1300 4300
-NoConn ~ 3750 4350
 Wire Wire Line
 	1000 3150 1000 3350
 Wire Wire Line
 	1400 1750 1400 3450
+Wire Wire Line
+	1300 5100 900  5100
+Wire Wire Line
+	1300 5000 1300 5100
+Wire Wire Line
+	1300 5100 1300 5200
+Connection ~ 1300 5100
+Wire Wire Line
+	900  2550 900  5100
+Wire Wire Line
+	900  5100 900  6700
+Connection ~ 900  5100
+Wire Wire Line
+	3750 4350 3800 4350
+Wire Wire Line
+	3800 4350 3800 4250
+Wire Wire Line
+	3750 4250 3800 4250
+Connection ~ 3800 4250
+Wire Wire Line
+	3800 4250 3850 4250
+$Comp
+L ARDUINO_PRO_MINI:ARDUINO_PRO_MINI U1
+U 1 1 60F56053
+P 3050 5350
+F 0 "U1" H 3050 6717 50  0000 C CNN
+F 1 "ARDUINO_PRO_MINI" H 3050 6626 50  0000 C CNN
+F 2 "3216LED:MODULE_ARDUINO_PRO_MINI" H 3050 5350 50  0001 L BNN
+F 3 "" H 3050 5350 50  0001 L BNN
+F 4 "Manufacturer Recommendations" H 3050 5350 50  0001 L BNN "STANDARD"
+F 5 "N/A" H 3050 5350 50  0001 L BNN "MAXIMUM_PACKAGE_HEIGHT"
+F 6 "SparkFun Electronics" H 3050 5350 50  0001 L BNN "MANUFACTURER"
+F 7 "N/A" H 3050 5350 50  0001 L BNN "PARTREV"
+	1    3050 5350
+	1    0    0    -1
+$EndComp
+Wire Wire Line
+	3750 6450 3750 6350
+Connection ~ 3750 6250
+Connection ~ 3750 6350
+Wire Wire Line
+	3750 6350 3750 6250
 $EndSCHEMATC
